Commit message: update yam mesh asset paths

File: i2rt/robot_models/yam/yam.urdf (robot description, URDF)
Before this commit: robot yam_v0, 7 links, 6 joints
Links:
- link base_link: geometry collision mesh filename=./assets/base_link_collision.stl; visual mesh filename=./assets/base_link_visual.stl
- link link_1: geometry collision mesh filename=./assets/link_1_collision.stl; visual mesh filename=./assets/link_1_visual.stl
- link link_2: geometry collision mesh filename=./assets/link_2_collision.stl; visual mesh filename=./assets/link_2_visual.stl
- link link_3: geometry collision mesh filename=./assets/link_3_collision.stl; visual mesh filename=./assets/link_3_visual.stl
- link link_4: geometry collision mesh filename=./assets/link_4_collision.stl; visual mesh filename=./assets/link_4_visual.stl
- link link_5: geometry collision mesh filename=./assets/link_5_collision.stl; visual mesh filename=./assets/link_5_visual.stl
- link link_6: geometry collision mesh filename=./assets/link_6_collision.stl; visual mesh filename=./assets/link_6_visual.stl
